File: fm/Underside.kicad_pcb (KiCad board)
At the start: 2 copper layers, 90 x 59 mm, 7 parts, among them J1 Micro_SD_Card_Det_Hirose_DM3AT, J2 Conn_01x04_Pin, U2 URM-37, U3 SeeeduinoXIAO

Commit message: reset
Routing:
- net GND: track 89.3 -> 92.3 mm
Changed lines of the file:
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@@
+	)
+	(gr_rect
+		(start 160.35 91.5)
+		(end 175.35 112.5)
+		(stroke
+			(width 0.1)
+			(type solid)
+		)
+		(fill no)
+		(layer "B.SilkS")
 	)
 	(gr_rect
@@
 	)
 	(gr_rect
-		(start 160.35 91.5)
-		(end 175.35 112.5)
-		(stroke
-			(width 0.1)
-			(type solid)
-		)
-		(fill no)
-		(layer "B.SilkS")
-	)
-	(gr_rect
 		(start 96 59)
 		(end 186 118)
@@
 		(start 152.54 69.04)
 		(end 155 69.04)
-		(width 0.2)
+		(width 0.6)
 		(layer "F.Cu")
 		(net 9)
@@
 	)
 	(segment
+		(start 157.96 69.04)
+		(end 158 69)
+		(width 0.2)
+		(layer "F.Cu")
+		(net 9)
+	)
+	(segment
 		(start 121.88 84.88)
 		(end 121.88 82.2)
@@
 		(layer "F.Cu")
 		(net 9)
+	)
+	(segment
+		(start 155 69.04)
+		(end 157.96 69.04)
+		(width 0.6)
+		(layer "F.Cu")
+		(net 9)

Commit message: re-production
Parts:
- added J3: Conn_01x04_Socket, Connector_PinSocket_2.54mm:PinSocket_1x04_P2.54mm_Vertical, F.Cu at (121.9, 114.3)
- J2: value Conn_01x04_Pin -> Conn_01x03_Socket; footprint TORICA_Hardwarelib_self-made:PA_Connector_Post_4Pin -> Connector_JST:JST_PH_S3B-PH-K_1x03_P2.00mm_Horizontal
- moved J1 5.12 mm to (116.8, 80.0)
- moved U2 4.65 mm to (126.9, 88.7)
- moved U3 4.27 mm to (146.5, 69.8)
- moved Under_URAT1 4.15 mm to (169.7, 71.1)
- moved J2 3.77 mm to (168.2, 81.4), turned to 0 degrees
Connections:
- J2 pad 1: Net-(J2-Pin_1) -> GND
- J2 pad 3: GND -> +3.3V
- U3 pad 4: unconnected-(U3-PA11_A3_D3-Pad4) -> Net-(J2-Pin_2)
- U3 pad 5: Net-(J2-Pin_1) -> /SDI
- U3 pad 6: Net-(J2-Pin_2) -> /SCK
- Under_URAT1 pad 2: +5V -> /PRXT
- Under_URAT1 pad 4: /PRXT -> +5V
Routing:
- net +3.3V: track 78.7 -> 230.0 mm, vias 0 -> 2
- net GND: track 92.3 -> 5.72 mm, vias 4 -> 56
- net Net-(U2-ECHO): track 105.2 -> 33.5 mm
- net /SDI: track 0.00 -> 61.7 mm, vias 0 -> 1
- net /SCK: track 0.00 -> 56.6 mm
- net Net-(U2-COMP/TRIG): track 80.0 -> 35.3 mm, vias 0 -> 2
- net Net-(J2-Pin_1): track 28.2 -> 0.00 mm, vias 2 -> 0
- net Net-(J1-CLK): track 37.7 -> 61.3 mm, vias 2 -> 1
- net /PTXR: track 37.4 -> 18.0 mm
- net /CS: track 33.1 -> 40.8 mm, vias 0 -> 1
- net Net-(J1-DAT0): track 34.0 -> 39.9 mm, vias 2 -> 1
- net +5V: track 14.2 -> 19.7 mm
- net Net-(J1-CMD): track 47.7 -> 52.6 mm, vias 2 -> 1
- net /PRXT: track 38.2 -> 42.8 mm
- net Net-(J2-Pin_2): track 48.6 -> 47.4 mm, vias 1 -> 0
- added copper zone on B.Cu, net GND
