File: fm/Underside.kicad_sch (KiCad schematic)
At the start: 5 parts, among them J1 Micro_SD_Card_Det_Hirose_DM3AT, J2 Conn_01x04_Pin, U2 URM-37, U3 SeeeduinoXIAO

Commit message: re-production
Parts:
- added J3: Conn_01x04_Socket, Connector_PinSocket_2.54mm:PinSocket_1x04_P2.54mm_Vertical, symbol Connector:Conn_01x04_Socket
- J2: value Conn_01x04_Pin -> Conn_01x03_Socket; footprint TORICA_Hardwarelib_self-made:PA_Connector_Post_4Pin -> Connector_JST:JST_PH_S3B-PH-K_1x03_P2.00mm_Horizontal; symbol Connector:Conn_01x04_Pin -> Connector:Conn_01x03_Socket
Connections:
- net +3.3V: now also J2.3 (Pin_3), J3.1 (Pin_1); no longer J2.4 (Pin_4)
- net +5V: now also Under_URAT1.4 (Pin_4); no longer Under_URAT1.2 (Pin_2)
- net GND: now also J2.1 (Pin_1), J3.2 (Pin_2); no longer J2.3 (Pin_3)
- net PRXT: now also Under_URAT1.2 (Pin_2); no longer Under_URAT1.4 (Pin_4)
- net at U3.4 (PA11_A3_D3): now also J2.2 (Pin_2)
- net SDI: now reaches U3.5 (PA8_A4_D4_SDA)
- net SDI: now also J3.4 (Pin_4); no longer J2.1 (Pin_1)
- net SCK: now reaches U3.6 (PA9_A5_D5_SCL)
- net SCK: now also J3.3 (Pin_3); no longer J2.2 (Pin_2)
- no-connect marks 11 -> 10
